Commit message: add basic end effector

File: src/ur_description_custom/urdf/ur.urdf.xacro (robot description, xacro)
@@ -85,4 +85,10 @@
      <origin xyz="0 0 0" rpy="0 0 0" />          <!-- position robot in the world -->
    </xacro:ur_robot>
+   <xacro:include filename="$(find ur_description_custom)/urdf/end_eff_basic.xacro"/>
+   <joint name="tool0_to_end_eff" type="fixed">
+    <parent link="$(arg tf_prefix)tool0"/>
+    <child link="end_eff_base_link"/>
+    <origin xyz="0 0.02 0.02" rpy="0 0 0"/>
+   </joint>
    <xacro:if value="$(arg sim_gazebo)">
     <!-- Gazebo plugins -->

Commit message: rotate end effector

File: src/ur_description_custom/urdf/ur.urdf.xacro (robot description, xacro)
@@ -89,5 +89,5 @@
     <parent link="$(arg tf_prefix)tool0"/>
     <child link="end_eff_base_link"/>
-    <origin xyz="0 0.02 0.02" rpy="0 0 0"/>
+    <origin xyz="-0.02 0 0.02" rpy="0 0 1.5708"/>
    </joint>
    <xacro:if value="$(arg sim_gazebo)">

Commit message: add new end effector

File: src/ur_description_custom/urdf/ur.urdf.xacro (robot description, xacro)
@@ -85,9 +85,15 @@
      <origin xyz="0 0 0" rpy="0 0 0" />          <!-- position robot in the world -->
    </xacro:ur_robot>
-   <xacro:include filename="$(find ur_description_custom)/urdf/end_eff_basic.xacro"/>
+   <!-- <xacro:include filename="$(find ur_description_custom)/urdf/end_eff_basic.xacro"/>
    <joint name="tool0_to_end_eff" type="fixed">
     <parent link="$(arg tf_prefix)tool0"/>
     <child link="end_eff_base_link"/>
     <origin xyz="-0.02 0 0.02" rpy="0 0 1.5708"/>
+   </joint> -->
+   <xacro:include filename="$(find ur_description_custom)/urdf/end_eff_detailed.xacro"/>
+   <joint name="tool0_to_end_eff" type="fixed">
+    <parent link="$(arg tf_prefix)tool0"/>
+    <child link="$(arg tf_prefix)end_eff_base_link"/>
+    <origin xyz="-0.2 0.38 0.18" rpy="-1.5708 0 -1.5708"/>
    </joint>
    <xacro:if value="$(arg sim_gazebo)">

Commit message: add tf support for movement actions

File: src/ur_description_custom/urdf/ur.urdf.xacro (robot description, xacro)
@@ -102,5 +102,5 @@
     <parent link="$(arg tf_prefix)tool0"/>
     <child link="$(arg tf_prefix)end_eff_contact"/>
-    <origin xyz="0.0 0.2 0.18" rpy="0 0 0"/>
+    <origin xyz="0.0 0.2 0.18" rpy="0 3.1416 -1.5708"/>
    </joint>
    <xacro:if value="$(arg sim_gazebo)">

File: src/ur_moveit_config_custom/srdf/ur_macro.srdf.xacro (robot description, xacro)
@@ -16,26 +16,10 @@
     <!--GROUP STATES - Purpose - Define a named state for a particular group, in terms of joint values. This is useful to define states like 'folded arms'-->
     <group_state name="${prefix}home" group="${prefix}${name}_manipulator">
-      <joint name="${prefix}elbow_joint" value="0" />
+      <joint name="${prefix}elbow_joint" value="1.5707" />
       <joint name="${prefix}shoulder_lift_joint" value="-1.5707" />
-      <joint name="${prefix}shoulder_pan_joint" value="0" />
-      <joint name="${prefix}wrist_1_joint" value="0" />
-      <joint name="${prefix}wrist_2_joint" value="0" />
+      <joint name="${prefix}shoulder_pan_joint" value="0.8" />
+      <joint name="${prefix}wrist_1_joint" value="-1.5707" />
+      <joint name="${prefix}wrist_2_joint" value="-1.5707" />
       <joint name="${prefix}wrist_3_joint" value="0" />
-    </group_state>
-    <group_state name="${prefix}up" group="${prefix}${name}_manipulator">
-      <joint name="${prefix}elbow_joint" value="0" />
-      <joint name="${prefix}shoulder_lift_joint" value="-1.5707" />
-      <joint name="${prefix}shoulder_pan_joint" value="0" />
-      <joint name="${prefix}wrist_1_joint" value="-1.5707" />
-      <joint name="${prefix}wrist_2_joint" value="0" />
-      <joint name="${prefix}wrist_3_joint" value="0" />
-    </group_state>
-    <group_state name="${prefix}test_configuration" group="${prefix}${name}_manipulator">
-      <joint name="${prefix}elbow_joint" value="1.4" />
-      <joint name="${prefix}shoulder_lift_joint" value="-1.62" />
-      <joint name="${prefix}shoulder_pan_joint" value="1.54" />
-      <joint name="${prefix}wrist_1_joint" value="-1.2" />
-      <joint name="${prefix}wrist_2_joint" value="-1.6" />
-      <joint name="${prefix}wrist_3_joint" value="-0.11" />
     </group_state>
     <!--END EFFECTOR - Purpose - Represent information about an end effector.-->

Commit message: tune end effector dimensions

File: src/ur_description_custom/urdf/ur.urdf.xacro (robot description, xacro)
@@ -95,5 +95,5 @@
     <parent link="$(arg tf_prefix)tool0"/>
     <child link="$(arg tf_prefix)end_eff_base_link"/>
-    <origin xyz="0 0 0" rpy="0 0 0"/>
+    <origin xyz="0 0 0" rpy="0 0 3.1416"/>
    </joint>
    <!-- End effector contact point frame -->
@@ -102,5 +102,5 @@
     <parent link="$(arg tf_prefix)tool0"/>
     <child link="$(arg tf_prefix)end_eff_contact"/>
-    <origin xyz="0.0 0.15 0.14" rpy="0 3.1416 -1.5708"/>
+    <origin xyz="0.0 -0.137 0.14" rpy="0 3.1416 1.5708"/>
    </joint>
    <xacro:if value="$(arg sim_gazebo)">
