Commit message: align moveit with end effector

File: src/ur_description_custom/urdf/end_eff_detailed.xacro (robot description, xacro)
@@ -1,5 +1,6 @@
 <?xml version="1.0"?>
 <robot xmlns:xacro="http://www.ros.org/wiki/xacro">
-  <link name="end_eff_base_link">
+  <xacro:arg name="tf_prefix" default=""/>
+  <link name="$(arg tf_prefix)end_eff_base_link">
     <visual>
       <geometry>

File: src/ur_description_custom/urdf/ur.urdf.xacro (robot description, xacro)
@@ -97,4 +97,11 @@
     <origin xyz="-0.2 0.38 0.18" rpy="-1.5708 0 -1.5708"/>
    </joint>
+   <!-- End effector contact point frame -->
+   <link name="$(arg tf_prefix)end_eff_contact"/>
+   <joint name="tool0_to_end_eff_contact" type="fixed">
+    <parent link="$(arg tf_prefix)tool0"/>
+    <child link="$(arg tf_prefix)end_eff_contact"/>
+    <origin xyz="0.0 0.2 0.18" rpy="0 0 0"/>
+   </joint>
    <xacro:if value="$(arg sim_gazebo)">
     <!-- Gazebo plugins -->

Commit message: update end eff urdf

File: src/ur_description_custom/urdf/end_eff_detailed.xacro (robot description, xacro)
@@ -4,4 +4,5 @@
   <link name="$(arg tf_prefix)end_eff_base_link">
     <visual>
+      <origin xyz="-1.077 0.155 0.15" rpy="-1.5707 0 -1.5707"/>
       <geometry>
         <mesh filename="package://ur_description_custom/meshes/end_eff/assembly.stl" scale="0.001 0.001 0.001"/>

File: src/ur_description_custom/urdf/ur.urdf.xacro (robot description, xacro)
@@ -95,5 +95,5 @@
     <parent link="$(arg tf_prefix)tool0"/>
     <child link="$(arg tf_prefix)end_eff_base_link"/>
-    <origin xyz="-0.2 0.38 0.18" rpy="-1.5708 0 -1.5708"/>
+    <origin xyz="0 0 0" rpy="0 0 0"/>
    </joint>
    <!-- End effector contact point frame -->
@@ -102,5 +102,5 @@
     <parent link="$(arg tf_prefix)tool0"/>
     <child link="$(arg tf_prefix)end_eff_contact"/>
-    <origin xyz="0.0 0.2 0.18" rpy="0 3.1416 -1.5708"/>
+    <origin xyz="0.0 0.15 0.14" rpy="0 3.1416 -1.5708"/>
    </joint>
    <xacro:if value="$(arg sim_gazebo)">

Commit message: fix end eff height in model

File: src/ur_description_custom/urdf/end_eff_detailed.xacro (robot description, xacro)
@@ -4,5 +4,5 @@
   <link name="$(arg tf_prefix)end_eff_base_link">
     <visual>
-      <origin xyz="-1.077 0.155 0.15" rpy="-1.5707 0 -1.5707"/>
+      <origin xyz="-1.077 0.155 0.172" rpy="-1.5707 0 -1.5707"/>
       <geometry>
         <mesh filename="package://ur_description_custom/meshes/end_eff/assembly.stl" scale="0.001 0.001 0.001"/>

File: src/ur_description_custom/urdf/ur.urdf.xacro (robot description, xacro)
@@ -102,5 +102,5 @@
     <parent link="$(arg tf_prefix)tool0"/>
     <child link="$(arg tf_prefix)end_eff_contact"/>
-    <origin xyz="0.0 -0.137 0.14" rpy="0 3.1416 1.5708"/>
+    <origin xyz="0.0 -0.137 0.162" rpy="0 3.1416 1.5708"/>
    </joint>
    <xacro:if value="$(arg sim_gazebo)">
